Commit message: upload_sans for test

File: robot_urdf/10_0_4_10_11_5_9_6_13_7_3_6_14_0_8_2/10_0_4_10_11_5_9_6_13_7_3_6_14_0_8_2.urdf (robot description, URDF)
Before this commit: robot mod_test, 21 links, 20 joints
Links:
- link 101: geometry collision mesh filename=package://meshes/module4.STL; visual mesh filename=package://meshes/module4.STL
- link 102: geometry collision mesh filename=package://meshes/module10.STL; visual mesh filename=package://meshes/module10.STL
- link 111: geometry collision mesh filename=package://meshes/module9.STL; visual mesh filename=package://meshes/module9.STL
- link 112: geometry collision mesh filename=package://meshes/module6.STL; visual mesh filename=package://meshes/module6.STL
- link 131: geometry collision mesh filename=package://meshes/module3.STL; visual mesh filename=package://meshes/module3.STL
- link 132: geometry collision mesh filename=package://meshes/module6.STL; visual mesh filename=package://meshes/module6.STL
- link 141: geometry collision mesh filename=package://meshes/module8.STL; visual mesh filename=package://meshes/module8.STL
- link 142: geometry collision mesh filename=package://meshes/module2.STL; visual mesh filename=package://meshes/module2.STL
Joints:
- removed joint 103_ball2
- removed joint 113_ball1
- removed joint 133_ball4
- removed joint 143_ball3
- added joint 103_ball1: type fixed, parent 103, child ball_1, origin xyz=0.0612 -0.13431 0 rpy=0 0 0, axis 0 0 0
- added joint 113_ball2: type fixed, parent 113, child ball_2, origin xyz=0.0612 -0.13431 0 rpy=0 0 0, axis 0 0 0
- added joint 133_ball3: type fixed, parent 133, child ball_3, origin xyz=0.0612 -0.13431 0 rpy=0 0 0, axis 0 0 0
- added joint 143_ball4: type fixed, parent 143, child ball_4, origin xyz=0.0612 -0.13431 0 rpy=0 0 0, axis 0 0 0
- joint 101_102: origin xyz=0.0816 0 0 rpy=4.712389 0 0 -> xyz=0.0816 0 0 rpy=2.094395 0 0
- joint 102_103: origin xyz=0.0816 0 0 rpy=1.047198 0 0 -> xyz=0.0816 0 0 rpy=5.235988 0 0
- joint 111_112: origin xyz=0.0816 0 0 rpy=1.047198 0 0 -> xyz=0.0816 0 0 rpy=4.712389 0 0
- joint 112_113: origin xyz=0.0816 0 0 rpy=0.000000 0 0 -> xyz=0.0816 0 0 rpy=3.141593 0 0
- joint 131_132: origin xyz=0.0816 0 0 rpy=5.235988 0 0 -> xyz=0.0816 0 0 rpy=1.570796 0 0
- joint 132_133: origin xyz=0.0816 0 0 rpy=0.000000 0 0 -> xyz=0.0816 0 0 rpy=3.141593 0 0
- joint 141_142: origin xyz=0.0816 0 0 rpy=1.570796 0 0 -> xyz=0.0816 0 0 rpy=4.188790 0 0
- joint 142_143: origin xyz=0.0816 0 0 rpy=5.235988 0 0 -> xyz=0.0816 0 0 rpy=1.047198 0 0
- joint body_110: origin xyz=0.083523 0.027138 -0.016769 rpy=3.141593 -1.382126 0.314159 -> xyz=0.083523 0.027138 -0.016769 rpy=-1.935587 1.017234 -1.570734
- joint body_130: origin xyz=-0.083523 0.027138 -0.016769 rpy=3.141593 -1.382126 2.827433 -> xyz=-0.083523 0.027138 -0.016769 rpy=1.935587 1.017234 -1.570859
